File: pcb/single_buckpuck_channel.sch (KiCad schematic (older format))
At the start: 4 parts, among them P12 CurrentOutput

Commit message: Initial changes for version-3 design
Parts:
- removed B4: CURRENT_SENSOR_BOARD, symbol CURRENT_SENSOR_BOARD
Connections:
- net labels added: Control, LED+, LED-, Potentiometer
- net labels removed: CurrentSense, IP+, IP-, PotentiometerInput+, PotentiometerInputWiper, PotentiometerOutput
- wire segments 28 -> 16
- no-connect marks 0 -> 1
Changed lines of the file:
@@
-EESchema Schematic File Version 2  date Wed 08 Jun 2011 02:44:18 PM PDT
+EESchema Schematic File Version 2  date Mon 11 Jul 2011 09:22:36 PM PDT
 LIBS:power
 LIBS:device
@@
 Sheet 5 5
 Title "Single Buckpuck Channel"
-Date "8 jun 2011"
-Rev "2.0"
+Date "12 jul 2011"
+Rev "3.0"
 Comp ""
 Comment1 ""
@@
 Comment4 ""
 $EndDescr
-Text Label 5400 3500 0    60   ~ 0
-IP-
-Text Label 5250 3000 0    60   ~ 0
-IP+
+NoConn ~ 4900 4000
+Text Label 5150 3650 0    60   ~ 0
+LED-
+Text Label 5150 3500 0    60   ~ 0
+LED+
 Wire Wire Line
-	6200 2900 6500 2900
+	5100 3500 5650 3500
 Wire Wire Line
-	6500 2900 6500 2750
+	7050 3800 7050 3950
 Wire Wire Line
-	6200 3000 6400 3000
+	7050 3950 7250 3950
 Wire Wire Line
-	5100 3500 5250 3500
+	7600 4250 7500 4250
 Wire Wire Line
-	5250 3500 5250 2900
-Wire Wire Line
-	5250 2900 5400 2900
-Wire Wire Line
-	4550 4400 4700 4400
-Wire Wire Line
-	4700 4400 4700 4000
-Wire Wire Line
-	7900 4050 7900 3950
-Wire Wire Line
-	7900 3950 7750 3950
-Connection ~ 5400 3700
-Wire Wire Line
-	5400 3850 5400 3650
-Wire Wire Line
-	4250 3200 4250 3500
-Wire Wire Line
-	4250 3500 4400 3500
-Wire Wire Line
-	4400 3800 4250 3800
-Wire Wire Line
-	4250 3800 4250 4100
-Wire Wire Line
-	5400 3650 5100 3650
+	7500 4250 7500 4100
 Wire Wire Line
 	5650 3700 5400 3700
 Wire Wire Line
-	7500 4100 7500 4250
+	5100 3650 5400 3650
 Wire Wire Line
-	7500 4250 7600 4250
+	4250 4100 4250 3800
 Wire Wire Line
-	7250 3950 7050 3950
+	4250 3800 4400 3800
 Wire Wire Line
-	7050 3950 7050 3800
+	4400 3500 4250 3500
 Wire Wire Line
-	4900 4000 4900 4400
+	4250 3500 4250 3200
 Wire Wire Line
-	4900 4400 5000 4400
+	5400 3650 5400 3700
 Wire Wire Line
-	5400 3100 5350 3100
+	7750 3950 7900 3950
 Wire Wire Line
-	5350 3100 5350 3500
+	7900 3950 7900 4050
 Wire Wire Line
-	5350 3500 5650 3500
+	4700 4000 4700 4400
 Wire Wire Line
-	6200 3100 6500 3100
-Wire Wire Line
-	6500 3100 6500 3200
-$Comp
-L GND #PWR028
-U 1 1 4DEEBBB6
-P 6500 3200
-AR Path="/4DEEDDA4/4DEEBBB6" Ref="#PWR028"  Part="1"
-AR Path="/4DEEDD9B/4DEEBBB6" Ref="#PWR034"  Part="1"
-AR Path="/4DEEDD8F/4DEEBBB6" Ref="#PWR040"  Part="1"
-AR Path="/4DEEDD29/4DEEBBB6" Ref="#PWR046"  Part="1"
-F 0 "#PWR046" H 6500 3200 30  0001 C CNN
-F 1 "GND" H 6500 3130 30  0001 C CNN
-	1    6500 3200
-	1    0    0    -1
-$EndComp
-$Comp
-L +5V #PWR029
-U 1 1 4DEEBBAF
-P 6500 2750
-AR Path="/4DEEDDA4/4DEEBBAF" Ref="#PWR029"  Part="1"
-AR Path="/4DEEDD9B/4DEEBBAF" Ref="#PWR035"  Part="1"
-AR Path="/4DEEDD8F/4DEEBBAF" Ref="#PWR041"  Part="1"
-AR Path="/4DEEDD29/4DEEBBAF" Ref="#PWR047"  Part="1"
-F 0 "#PWR047" H 6500 2840 20  0001 C CNN
-F 1 "+5V" H 6500 2840 30  0000 C CNN
-	1    6500 2750
-	1    0    0    -1
-$EndComp
-$Comp
-L CURRENT_SENSOR_BOARD B4
-U 1 1 4DEEBB77
-P 5800 3000
-AR Path="/4DEEDDA4/4DEEBB77" Ref="B4"  Part="1"
-AR Path="/4DEEDD9B/4DEEBB77" Ref="B3"  Part="1"
-AR Path="/4DEEDD8F/4DEEBB77" Ref="B2"  Part="1"
-AR Path="/4DEEDD29/4DEEBB77" Ref="B1"  Part="1"
-F 0 "B1" H 5800 2800 60  0000 C CNN
-F 1 "CURRENT_SENSOR_BOARD" H 5800 3250 60  0000 C CNN
-	1    5800 3000
-	1    0    0    -1
-$EndComp
-Text HLabel 5000 4400 2    60   Output ~ 0
-PotentiometerInput+
+	4700 4400 4550 4400
 Text HLabel 4550 4400 0    60   Input ~ 0
-PotentiometerInputWiper
+Control
 Text HLabel 7600 4250 2    60   Output ~ 0
-PotentiometerOutput
+Potentiometer
 $Comp
 L GND #PWR030
@@
 AR Path="/4DEEDD8F/4DD1EC8D" Ref="#PWR042"  Part="1"
 AR Path="/4DEEDD29/4DD1EC8D" Ref="#PWR048"  Part="1"
+AR Path="/4E1B87B2/4DD1EC8D" Ref="#PWR048"  Part="1"
+AR Path="/4E1B8863/4DD1EC8D" Ref="#PWR048"  Part="1"
 F 0 "#PWR048" H 7900 4050 30  0001 C CNN
 F 1 "GND" H 7900 3980 30  0001 C CNN
@@
 AR Path="/4DEEDD8F/4DD1EC8A" Ref="#PWR043"  Part="1"
 AR Path="/4DEEDD29/4DD1EC8A" Ref="#PWR049"  Part="1"
+AR Path="/4E1B87B2/4DD1EC8A" Ref="#PWR049"  Part="1"
+AR Path="/4E1B8863/4DD1EC8A" Ref="#PWR049"  Part="1"
 F 0 "#PWR049" H 7050 3890 20  0001 C CNN
 F 1 "+5V" H 7050 3890 30  0000 C CNN
@@
 AR Path="/4DEEDD8F/4DD1EC78" Ref="RV2"  Part="1"
 AR Path="/4DEEDD29/4DD1EC78" Ref="RV1"  Part="1"
+AR Path="/4E1B87B2/4DD1EC78" Ref="RV1"  Part="1"
+AR Path="/4E1B8863/4DD1EC78" Ref="RV1"  Part="1"
 F 0 "RV1" H 7500 3850 50  0000 C CNN
 F 1 "POT" H 7500 3950 50  0000 C CNN
@@
 	-1   0    0    1
 $EndComp
-Text HLabel 6400 3000 2    60   Output ~ 0
-CurrentSense
 $Comp
 L BUCKPUCK BP4
@@
 AR Path="/4DEEDD8F/4DD1A2DC" Ref="BP2"  Part="1"
 AR Path="/4DEEDD29/4DD1A2DC" Ref="BP1"  Part="1"
+AR Path="/4E1B87B2/4DD1A2DC" Ref="BP1"  Part="1"
+AR Path="/4E1B8863/4DD1A2DC" Ref="BP1"  Part="1"
 F 0 "BP1" H 5100 3450 60  0000 C CNN
 F 1 "BUCKPUCK" H 4750 3950 60  0000 C CNN
@@
 AR Path="/4DEEDD8F/4DD1A2DB" Ref="#PWR29"  Part="1"
 AR Path="/4DEEDD29/4DD1A2DB" Ref="#PWR22"  Part="1"
+AR Path="/4E1B87B2/4DD1A2DB" Ref="#PWR22"  Part="1"
+AR Path="/4E1B8863/4DD1A2DB" Ref="#PWR22"  Part="1"
 F 0 "#PWR22" H 4250 3260 30  0001 C CNN
 F 1 "VAA" H 4250 3310 30  0000 C CNN
@@
 AR Path="/4DEEDD8F/4DD1A2DA" Ref="#PWR044"  Part="1"
 AR Path="/4DEEDD29/4DD1A2DA" Ref="#PWR050"  Part="1"
+AR Path="/4E1B87B2/4DD1A2DA" Ref="#PWR050"  Part="1"
+AR Path="/4E1B8863/4DD1A2DA" Ref="#PWR050"  Part="1"
 F 0 "#PWR050" H 4250 4100 30  0001 C CNN
 F 1 "GND" H 4250 4030 30  0001 C CNN
@@
 AR Path="/4DEEDD8F/4DD1A2D9" Ref="P10"  Part="1"
 AR Path="/4DEEDD29/4DD1A2D9" Ref="P9"  Part="1"
+AR Path="/4E1B87B2/4DD1A2D9" Ref="P9"  Part="1"
+AR Path="/4E1B8863/4DD1A2D9" Ref="P9"  Part="1"
 F 0 "P9" V 5950 3600 40  0000 C CNN
 F 1 "CurrentOutput" V 6050 3600 40  0000 C CNN
@@
 	1    0    0    -1
 $EndComp
-$Comp
-L GND #PWR033
-U 1 1 4DD1A2D8
-P 5400 3850
-AR Path="/4DEEDDA4/4DD1A2D8" Ref="#PWR033"  Part="1"
-AR Path="/4DEEDD9B/4DD1A2D8" Ref="#PWR039"  Part="1"
-AR Path="/4DEEDD8F/4DD1A2D8" Ref="#PWR045"  Part="1"
-AR Path="/4DEEDD29/4DD1A2D8" Ref="#PWR051"  Part="1"
-F 0 "#PWR051" H 5400 3850 30  0001 C CNN
-F 1 "GND" H 5400 3780 30  0001 C CNN
-	1    5400 3850
-	1    0    0    -1
-$EndComp

Commit message: Finished schematic version 3
Changed lines of the file:
@@
-EESchema Schematic File Version 2  date Mon 11 Jul 2011 09:22:36 PM PDT
+EESchema Schematic File Version 2  date Tue 12 Jul 2011 03:30:38 PM PDT
 LIBS:power
 LIBS:device
@@
 EELAYER END
 $Descr A4 11700 8267
-Sheet 5 5
+Sheet 4 5
 Title "Single Buckpuck Channel"
 Date "12 jul 2011"
@@
 AR Path="/4DEEDD8F/4DD1EC8D" Ref="#PWR042"  Part="1"
 AR Path="/4DEEDD29/4DD1EC8D" Ref="#PWR048"  Part="1"
-AR Path="/4E1B87B2/4DD1EC8D" Ref="#PWR048"  Part="1"
-AR Path="/4E1B8863/4DD1EC8D" Ref="#PWR048"  Part="1"
-F 0 "#PWR048" H 7900 4050 30  0001 C CNN
+AR Path="/4E1B87B2/4DD1EC8D" Ref="#PWR043"  Part="1"
+AR Path="/4E1B8863/4DD1EC8D" Ref="#PWR040"  Part="1"
+AR Path="/4E1B8870/4DD1EC8D" Ref="#PWR034"  Part="1"
+AR Path="/4E1B886D/4DD1EC8D" Ref="#PWR037"  Part="1"
+F 0 "#PWR043" H 7900 4050 30  0001 C CNN
 F 1 "GND" H 7900 3980 30  0001 C CNN
 	1    7900 4050
@@
 AR Path="/4DEEDD8F/4DD1EC8A" Ref="#PWR043"  Part="1"
 AR Path="/4DEEDD29/4DD1EC8A" Ref="#PWR049"  Part="1"
-AR Path="/4E1B87B2/4DD1EC8A" Ref="#PWR049"  Part="1"
-AR Path="/4E1B8863/4DD1EC8A" Ref="#PWR049"  Part="1"
-F 0 "#PWR049" H 7050 3890 20  0001 C CNN
+AR Path="/4E1B87B2/4DD1EC8A" Ref="#PWR044"  Part="1"
+AR Path="/4E1B8863/4DD1EC8A" Ref="#PWR041"  Part="1"
+AR Path="/4E1B8870/4DD1EC8A" Ref="#PWR035"  Part="1"
+AR Path="/4E1B886D/4DD1EC8A" Ref="#PWR038"  Part="1"
+F 0 "#PWR044" H 7050 3890 20  0001 C CNN
 F 1 "+5V" H 7050 3890 30  0000 C CNN
 	1    7050 3800
@@
 AR Path="/4DEEDD29/4DD1EC78" Ref="RV1"  Part="1"
 AR Path="/4E1B87B2/4DD1EC78" Ref="RV1"  Part="1"
-AR Path="/4E1B8863/4DD1EC78" Ref="RV1"  Part="1"
-F 0 "RV1" H 7500 3850 50  0000 C CNN
+AR Path="/4E1B8863/4DD1EC78" Ref="RV2"  Part="1"
+AR Path="/4E1B8870/4DD1EC78" Ref="RV3"  Part="1"
+AR Path="/4E1B886D/4DD1EC78" Ref="RV4"  Part="1"
+F 0 "RV3" H 7500 3850 50  0000 C CNN
 F 1 "POT" H 7500 3950 50  0000 C CNN
 	1    7500 3950
@@
 AR Path="/4DEEDD29/4DD1A2DC" Ref="BP1"  Part="1"
 AR Path="/4E1B87B2/4DD1A2DC" Ref="BP1"  Part="1"
-AR Path="/4E1B8863/4DD1A2DC" Ref="BP1"  Part="1"
-F 0 "BP1" H 5100 3450 60  0000 C CNN
+AR Path="/4E1B8863/4DD1A2DC" Ref="BP2"  Part="1"
+AR Path="/4E1B8870/4DD1A2DC" Ref="BP3"  Part="1"
+AR Path="/4E1B886D/4DD1A2DC" Ref="BP4"  Part="1"
+F 0 "BP3" H 5100 3450 60  0000 C CNN
 F 1 "BUCKPUCK" H 4750 3950 60  0000 C CNN
 	1    4750 3650
@@
 AR Path="/4DEEDD8F/4DD1A2DB" Ref="#PWR29"  Part="1"
 AR Path="/4DEEDD29/4DD1A2DB" Ref="#PWR22"  Part="1"
-AR Path="/4E1B87B2/4DD1A2DB" Ref="#PWR22"  Part="1"
-AR Path="/4E1B8863/4DD1A2DB" Ref="#PWR22"  Part="1"
-F 0 "#PWR22" H 4250 3260 30  0001 C CNN
+AR Path="/4E1B87B2/4DD1A2DB" Ref="#PWR32"  Part="1"
+AR Path="/4E1B8863/4DD1A2DB" Ref="#PWR36"  Part="1"
+AR Path="/4E1B8870/4DD1A2DB" Ref="#PWR44"  Part="1"
+AR Path="/4E1B886D/4DD1A2DB" Ref="#PWR40"  Part="1"
+F 0 "#PWR44" H 4250 3260 30  0001 C CNN
 F 1 "VAA" H 4250 3310 30  0000 C CNN
 	1    4250 3200
@@
 AR Path="/4DEEDD8F/4DD1A2DA" Ref="#PWR044"  Part="1"
 AR Path="/4DEEDD29/4DD1A2DA" Ref="#PWR050"  Part="1"
-AR Path="/4E1B87B2/4DD1A2DA" Ref="#PWR050"  Part="1"
-AR Path="/4E1B8863/4DD1A2DA" Ref="#PWR050"  Part="1"
-F 0 "#PWR050" H 4250 4100 30  0001 C CNN
+AR Path="/4E1B87B2/4DD1A2DA" Ref="#PWR045"  Part="1"
+AR Path="/4E1B8863/4DD1A2DA" Ref="#PWR042"  Part="1"
+AR Path="/4E1B8870/4DD1A2DA" Ref="#PWR036"  Part="1"
+AR Path="/4E1B886D/4DD1A2DA" Ref="#PWR039"  Part="1"
+F 0 "#PWR045" H 4250 4100 30  0001 C CNN
 F 1 "GND" H 4250 4030 30  0001 C CNN
 	1    4250 4100
@@
 AR Path="/4DEEDD29/4DD1A2D9" Ref="P9"  Part="1"
 AR Path="/4E1B87B2/4DD1A2D9" Ref="P9"  Part="1"
-AR Path="/4E1B8863/4DD1A2D9" Ref="P9"  Part="1"
-F 0 "P9" V 5950 3600 40  0000 C CNN
+AR Path="/4E1B8863/4DD1A2D9" Ref="P10"  Part="1"
+AR Path="/4E1B8870/4DD1A2D9" Ref="P11"  Part="1"
+AR Path="/4E1B886D/4DD1A2D9" Ref="P12"  Part="1"
+F 0 "P11" V 5950 3600 40  0000 C CNN
 F 1 "CurrentOutput" V 6050 3600 40  0000 C CNN
 	1    6000 3600

Commit message: Creating version-4
Parts:
- added U?: SSR_DC_6PIN, symbol SSR_DC_6PIN
Changed lines of the file:
@@
-EESchema Schematic File Version 2  date Thu 14 Jul 2011 12:12:51 PM PDT
+EESchema Schematic File Version 2  date Sun 31 Jul 2011 01:58:26 PM PDT
 LIBS:power
 LIBS:device
@@
 EELAYER END
 $Descr A4 11700 8267
-Sheet 4 5
+Sheet 5 5
 Title "Single Buckpuck Channel"
 Date "14 jul 2011"
@@
 Comment4 ""
 $EndDescr
+$Comp
+L SSR_DC_6PIN U?
+U 1 1 4E35C1C4
+P 3200 3350
+F 0 "U?" H 2950 3550 60  0000 C CNN
+F 1 "SSR_DC_6PIN" H 3200 3150 60  0000 C CNN
+	1    3200 3350
+	1    0    0    -1
+$EndComp
 NoConn ~ 4900 4000
 Text Label 5150 3650 0    60   ~ 0
@@
 AR Path="/4E1B8870/4DD1EC78" Ref="RV3"  Part="1"
 AR Path="/4E1B886D/4DD1EC78" Ref="RV4"  Part="1"
-F 0 "RV3" H 7500 3850 50  0000 C CNN
+F 0 "RV1" H 7500 3850 50  0000 C CNN
 F 1 "POT" H 7500 3950 50  0000 C CNN
 	1    7500 3950
@@
 AR Path="/4E1B8870/4DD1A2DC" Ref="BP3"  Part="1"
 AR Path="/4E1B886D/4DD1A2DC" Ref="BP4"  Part="1"
-F 0 "BP3" H 5100 3450 60  0000 C CNN
+F 0 "BP1" H 5100 3450 60  0000 C CNN
 F 1 "BUCKPUCK" H 4750 3950 60  0000 C CNN
 	1    4750 3650
@@
 AR Path="/4E1B8870/4DD1A2DB" Ref="#PWR44"  Part="1"
 AR Path="/4E1B886D/4DD1A2DB" Ref="#PWR40"  Part="1"
-F 0 "#PWR44" H 4250 3260 30  0001 C CNN
+F 0 "#PWR32" H 4250 3260 30  0001 C CNN
 F 1 "VAA" H 4250 3310 30  0000 C CNN
 	1    4250 3200
@@
 AR Path="/4E1B8870/4DD1A2D9" Ref="P11"  Part="1"
 AR Path="/4E1B886D/4DD1A2D9" Ref="P12"  Part="1"
-F 0 "P11" V 5950 3600 40  0000 C CNN
+F 0 "P9" V 5950 3600 40  0000 C CNN
 F 1 "CurrentOutput" V 6050 3600 40  0000 C CNN
 	1    6000 3600

Commit message: Made intial version-4 changes to the schematic
Connections:
- net GND: now also U?.2 (-CTL)
- net VAA: now also U?.4 (+LOAD), U?.6 (+LOAD); no longer BP4.5 (V+)
- net SSRControl: now reaches U?.1 (+CTL)
- net BuckpuckV+: now reaches U?.5 (-LOAD)
- net BuckpuckV+: now also BP4.5 (V+)
- net Control renamed BuckpuckControl
- no-connect marks 1 -> 2
Other:
- moved on the sheet: U?
Changed lines of the file:
@@
-EESchema Schematic File Version 2  date Sun 31 Jul 2011 01:58:26 PM PDT
+EESchema Schematic File Version 2  date Sun 31 Jul 2011 03:57:05 PM PDT
 LIBS:power
 LIBS:device
@@
 EELAYER END
 $Descr A4 11700 8267
-Sheet 5 5
+Sheet 4 3
 Title "Single Buckpuck Channel"
-Date "14 jul 2011"
+Date "31 jul 2011"
 Rev "3.0"
 Comp ""
@@
 Comment4 ""
 $EndDescr
+Text HLabel 1950 3400 0    60   Input ~ 0
+SSRControl
+Wire Wire Line
+	2300 3400 1950 3400
+Wire Wire Line
+	3600 3500 4400 3500
+Wire Wire Line
+	3600 3600 3750 3600
+Wire Wire Line
+	3750 3600 3750 3300
+Wire Wire Line
+	4550 4400 4700 4400
+Wire Wire Line
+	4700 4400 4700 4000
+Wire Wire Line
+	7900 4050 7900 3950
+Wire Wire Line
+	7900 3950 7750 3950
+Wire Wire Line
+	5400 3650 5400 3700
+Wire Wire Line
+	4400 3800 4250 3800
+Wire Wire Line
+	4250 3800 4250 4100
+Wire Wire Line
+	5400 3650 5100 3650
+Wire Wire Line
+	5400 3700 5650 3700
+Wire Wire Line
+	7500 4100 7500 4250
+Wire Wire Line
+	7500 4250 7600 4250
+Wire Wire Line
+	7250 3950 7050 3950
+Wire Wire Line
+	7050 3950 7050 3800
+Wire Wire Line
+	5100 3500 5650 3500
+Wire Wire Line
+	3600 3400 3750 3400
+Connection ~ 3750 3400
+Wire Wire Line
+	2300 3500 2100 3500
+Wire Wire Line
+	2100 3500 2100 3650
+$Comp
+L GND #PWR?
+U 1 1 4E35D6B2
+P 2100 3650
+AR Path="/4E1B87B2/4E35D6B2" Ref="#PWR?"  Part="1"
+AR Path="/4E1B8863/4E35D6B2" Ref="#PWR?"  Part="1"
+F 0 "#PWR?" H 2100 3650 30  0001 C CNN
+F 1 "GND" H 2100 3580 30  0001 C CNN
+	1    2100 3650
+	1    0    0    -1
+$EndComp
+Text Label 3800 3500 0    60   ~ 0
+BuckpuckV+
+NoConn ~ 2300 3600
 $Comp
 L SSR_DC_6PIN U?
 U 1 1 4E35C1C4
-P 3200 3350
-F 0 "U?" H 2950 3550 60  0000 C CNN
-F 1 "SSR_DC_6PIN" H 3200 3150 60  0000 C CNN
-	1    3200 3350
+P 2950 3500
+AR Path="/4E1B87B2/4E35C1C4" Ref="U?"  Part="1"
+AR Path="/4E1B8863/4E35C1C4" Ref="U?"  Part="1"
+F 0 "U?" H 2700 3700 60  0000 C CNN
+F 1 "SSR_DC_6PIN" H 2950 3300 60  0000 C CNN
+	1    2950 3500
 	1    0    0    -1
 $EndComp
@@
 Text Label 5150 3500 0    60   ~ 0
 LED+
-Wire Wire Line
-	5100 3500 5650 3500
-Wire Wire Line
-	7050 3800 7050 3950
-Wire Wire Line
-	7050 3950 7250 3950
-Wire Wire Line
-	7600 4250 7500 4250
-Wire Wire Line
-	7500 4250 7500 4100
-Wire Wire Line
-	5650 3700 5400 3700
-Wire Wire Line
-	5100 3650 5400 3650
-Wire Wire Line
-	4250 4100 4250 3800
-Wire Wire Line
-	4250 3800 4400 3800
-Wire Wire Line
-	4400 3500 4250 3500
-Wire Wire Line
-	4250 3500 4250 3200
-Wire Wire Line
-	5400 3650 5400 3700
-Wire Wire Line
-	7750 3950 7900 3950
-Wire Wire Line
-	7900 3950 7900 4050
-Wire Wire Line
-	4700 4000 4700 4400
-Wire Wire Line
-	4700 4400 4550 4400
 Text HLabel 4550 4400 0    60   Input ~ 0
-Control
+BuckpuckControl
 Text HLabel 7600 4250 2    60   Output ~ 0
 Potentiometer
@@
 AR Path="/4E1B8870/4DD1EC8D" Ref="#PWR034"  Part="1"
 AR Path="/4E1B886D/4DD1EC8D" Ref="#PWR037"  Part="1"
-F 0 "#PWR043" H 7900 4050 30  0001 C CNN
+F 0 "#PWR040" H 7900 4050 30  0001 C CNN
 F 1 "GND" H 7900 3980 30  0001 C CNN
 	1    7900 4050
@@
 AR Path="/4E1B8870/4DD1EC8A" Ref="#PWR035"  Part="1"
 AR Path="/4E1B886D/4DD1EC8A" Ref="#PWR038"  Part="1"
-F 0 "#PWR044" H 7050 3890 20  0001 C CNN
+F 0 "#PWR041" H 7050 3890 20  0001 C CNN
 F 1 "+5V" H 7050 3890 30  0000 C CNN
 	1    7050 3800
@@
 AR Path="/4E1B8870/4DD1EC78" Ref="RV3"  Part="1"
 AR Path="/4E1B886D/4DD1EC78" Ref="RV4"  Part="1"
-F 0 "RV1" H 7500 3850 50  0000 C CNN
+F 0 "RV2" H 7500 3850 50  0000 C CNN
 F 1 "POT" H 7500 3950 50  0000 C CNN
 	1    7500 3950
@@
 AR Path="/4E1B8870/4DD1A2DC" Ref="BP3"  Part="1"
 AR Path="/4E1B886D/4DD1A2DC" Ref="BP4"  Part="1"
-F 0 "BP1" H 5100 3450 60  0000 C CNN
+F 0 "BP2" H 5100 3450 60  0000 C CNN
 F 1 "BUCKPUCK" H 4750 3950 60  0000 C CNN
 	1    4750 3650
@@
 L VAA #PWR43
 U 1 1 4DD1A2DB
-P 4250 3200
+P 3750 3300
 AR Path="/4DEEDDA4/4DD1A2DB" Ref="#PWR43"  Part="1"
 AR Path="/4DEEDD9B/4DD1A2DB" Ref="#PWR36"  Part="1"
@@
 AR Path="/4E1B8870/4DD1A2DB" Ref="#PWR44"  Part="1"
 AR Path="/4E1B886D/4DD1A2DB" Ref="#PWR40"  Part="1"
-F 0 "#PWR32" H 4250 3260 30  0001 C CNN
-F 1 "VAA" H 4250 3310 30  0000 C CNN
-	1    4250 3200
+F 0 "#PWR36" H 3750 3360 30  0001 C CNN
+F 1 "VAA" H 3750 3410 30  0000 C CNN
+	1    3750 3300
 	1    0    0    -1
 $EndComp
@@
 AR Path="/4E1B8870/4DD1A2DA" Ref="#PWR036"  Part="1"
 AR Path="/4E1B886D/4DD1A2DA" Ref="#PWR039"  Part="1"
-F 0 "#PWR045" H 4250 4100 30  0001 C CNN
+F 0 "#PWR042" H 4250 4100 30  0001 C CNN
 F 1 "GND" H 4250 4030 30  0001 C CNN
 	1    4250 4100
@@
 AR Path="/4E1B8870/4DD1A2D9" Ref="P11"  Part="1"
 AR Path="/4E1B886D/4DD1A2D9" Ref="P12"  Part="1"
-F 0 "P9" V 5950 3600 40  0000 C CNN
+F 0 "P10" V 5950 3600 40  0000 C CNN
 F 1 "CurrentOutput" V 6050 3600 40  0000 C CNN
 	1    6000 3600
