File: pcb/single_buckpuck_channel.sch (KiCad schematic (older format))
At the start: 4 parts, among them P12 CurrentOutput

Commit message: Added IO expander to the schematic
Parts:
- added R?: R, symbol R
Connections:
- net BuckpuckControl renamed Buckpuck_Control
- net SSRControl: no longer names the net of U?.1 (+CTL)
- net SSRControl: now also R?.1
- new net SSR_Control: R?.2
Other:
- moved on the sheet: BP1, P9, RV1, U?
Changed lines of the file:
@@
-EESchema Schematic File Version 2  date Sun 31 Jul 2011 03:57:05 PM PDT
+EESchema Schematic File Version 2  date Tue 02 Aug 2011 06:03:40 PM PDT
 LIBS:power
 LIBS:device
@@
 EELAYER END
 $Descr A4 11700 8267
-Sheet 4 3
-Title "Single Buckpuck Channel"
-Date "31 jul 2011"
-Rev "3.0"
+Sheet 3 5
+Title "Buckpuck Current Controller"
+Date "3 aug 2011"
+Rev "4.0"
 Comp ""
 Comment1 ""
@@
 Comment4 ""
 $EndDescr
-Text HLabel 1950 3400 0    60   Input ~ 0
-SSRControl
-Wire Wire Line
-	2300 3400 1950 3400
-Wire Wire Line
-	3600 3500 4400 3500
-Wire Wire Line
-	3600 3600 3750 3600
-Wire Wire Line
-	3750 3600 3750 3300
-Wire Wire Line
-	4550 4400 4700 4400
-Wire Wire Line
-	4700 4400 4700 4000
-Wire Wire Line
-	7900 4050 7900 3950
-Wire Wire Line
-	7900 3950 7750 3950
-Wire Wire Line
-	5400 3650 5400 3700
-Wire Wire Line
-	4400 3800 4250 3800
-Wire Wire Line
-	4250 3800 4250 4100
-Wire Wire Line
-	5400 3650 5100 3650
-Wire Wire Line
-	5400 3700 5650 3700
-Wire Wire Line
-	7500 4100 7500 4250
-Wire Wire Line
-	7500 4250 7600 4250
-Wire Wire Line
-	7250 3950 7050 3950
-Wire Wire Line
-	7050 3950 7050 3800
-Wire Wire Line
-	5100 3500 5650 3500
-Wire Wire Line
-	3600 3400 3750 3400
-Connection ~ 3750 3400
-Wire Wire Line
-	2300 3500 2100 3500
-Wire Wire Line
-	2100 3500 2100 3650
+Wire Wire Line
+	2850 3800 2750 3800
+Wire Wire Line
+	4750 3900 5550 3900
+Wire Wire Line
+	4750 4000 4900 4000
+Wire Wire Line
+	4900 4000 4900 3700
+Wire Wire Line
+	5700 4800 5850 4800
+Wire Wire Line
+	5850 4800 5850 4400
+Wire Wire Line
+	9050 4450 9050 4350
+Wire Wire Line
+	9050 4350 8900 4350
+Wire Wire Line
+	6550 4050 6550 4100
+Wire Wire Line
+	5550 4200 5400 4200
+Wire Wire Line
+	5400 4200 5400 4500
+Wire Wire Line
+	6550 4050 6250 4050
+Wire Wire Line
+	6550 4100 6800 4100
+Wire Wire Line
+	8650 4500 8650 4650
+Wire Wire Line
+	8650 4650 8750 4650
+Wire Wire Line
+	8400 4350 8200 4350
+Wire Wire Line
+	8200 4350 8200 4200
+Wire Wire Line
+	6250 3900 6800 3900
+Wire Wire Line
+	4750 3800 4900 3800
+Connection ~ 4900 3800
+Wire Wire Line
+	3450 3900 3250 3900
+Wire Wire Line
+	3250 3900 3250 4050
+Wire Wire Line
+	3350 3800 3450 3800
+$Comp
+L R R?
+U 1 1 4E386D28
+P 3100 3800
+AR Path="/4E3873D3/4E386D28" Ref="R?"  Part="1"
+AR Path="/4E388079/4E386D28" Ref="R?"  Part="1"
+F 0 "R?" V 3180 3800 50  0000 C CNN
+F 1 "R" V 3100 3800 50  0000 C CNN
+	1    3100 3800
+	0    1    1    0
+$EndComp
+Text HLabel 2750 3800 0    60   Input ~ 0
+SSR_Control
 $Comp
 L GND #PWR?
 U 1 1 4E35D6B2
-P 2100 3650
+P 3250 4050
 AR Path="/4E1B87B2/4E35D6B2" Ref="#PWR?"  Part="1"
 AR Path="/4E1B8863/4E35D6B2" Ref="#PWR?"  Part="1"
-F 0 "#PWR?" H 2100 3650 30  0001 C CNN
-F 1 "GND" H 2100 3580 30  0001 C CNN
-	1    2100 3650
-	1    0    0    -1
-$EndComp
-Text Label 3800 3500 0    60   ~ 0
+AR Path="/4E3873D3/4E35D6B2" Ref="#PWR?"  Part="1"
+AR Path="/4E388079/4E35D6B2" Ref="#PWR?"  Part="1"
+F 0 "#PWR?" H 3250 4050 30  0001 C CNN
+F 1 "GND" H 3250 3980 30  0001 C CNN
+	1    3250 4050
+	1    0    0    -1
+$EndComp
+Text Label 4950 3900 0    60   ~ 0
 BuckpuckV+
-NoConn ~ 2300 3600
+NoConn ~ 3450 4000
 $Comp
 L SSR_DC_6PIN U?
 U 1 1 4E35C1C4
-P 2950 3500
+P 4100 3900
 AR Path="/4E1B87B2/4E35C1C4" Ref="U?"  Part="1"
 AR Path="/4E1B8863/4E35C1C4" Ref="U?"  Part="1"
-F 0 "U?" H 2700 3700 60  0000 C CNN
-F 1 "SSR_DC_6PIN" H 2950 3300 60  0000 C CNN
-	1    2950 3500
-	1    0    0    -1
-$EndComp
-NoConn ~ 4900 4000
-Text Label 5150 3650 0    60   ~ 0
+AR Path="/4E3873D3/4E35C1C4" Ref="U?"  Part="1"
+AR Path="/4E388079/4E35C1C4" Ref="U?"  Part="1"
+F 0 "U?" H 3850 4100 60  0000 C CNN
+F 1 "SSR_DC_6PIN" H 4100 3700 60  0000 C CNN
+	1    4100 3900
+	1    0    0    -1
+$EndComp
+NoConn ~ 6050 4400
+Text Label 6300 4050 0    60   ~ 0
 LED-
-Text Label 5150 3500 0    60   ~ 0
+Text Label 6300 3900 0    60   ~ 0
 LED+
-Text HLabel 4550 4400 0    60   Input ~ 0
-BuckpuckControl
-Text HLabel 7600 4250 2    60   Output ~ 0
+Text HLabel 5700 4800 0    60   Input ~ 0
+Buckpuck_Control
+Text HLabel 8750 4650 2    60   Output ~ 0
 Potentiometer
 $Comp
 L GND #PWR030
 U 1 1 4DD1EC8D
-P 7900 4050
+P 9050 4450
 AR Path="/4DEEDDA4/4DD1EC8D" Ref="#PWR030"  Part="1"
 AR Path="/4DEEDD9B/4DD1EC8D" Ref="#PWR036"  Part="1"
@@
 AR Path="/4E1B8870/4DD1EC8D" Ref="#PWR034"  Part="1"
 AR Path="/4E1B886D/4DD1EC8D" Ref="#PWR037"  Part="1"
-F 0 "#PWR040" H 7900 4050 30  0001 C CNN
-F 1 "GND" H 7900 3980 30  0001 C CNN
-	1    7900 4050
+AR Path="/4E3873D3/4DD1EC8D" Ref="#PWR043"  Part="1"
+AR Path="/4E388079/4DD1EC8D" Ref="#PWR043"  Part="1"
+F 0 "#PWR043" H 9050 4450 30  0001 C CNN
+F 1 "GND" H 9050 4380 30  0001 C CNN
+	1    9050 4450
 	1    0    0    -1
 $EndComp
@@
 L +5V #PWR031
 U 1 1 4DD1EC8A
-P 7050 3800
+P 8200 4200
 AR Path="/4DEEDDA4/4DD1EC8A" Ref="#PWR031"  Part="1"
 AR Path="/4DEEDD9B/4DD1EC8A" Ref="#PWR037"  Part="1"
@@
 AR Path="/4E1B8870/4DD1EC8A" Ref="#PWR035"  Part="1"
 AR Path="/4E1B886D/4DD1EC8A" Ref="#PWR038"  Part="1"
-F 0 "#PWR041" H 7050 3890 20  0001 C CNN
-F 1 "+5V" H 7050 3890 30  0000 C CNN
-	1    7050 3800
+AR Path="/4E3873D3/4DD1EC8A" Ref="#PWR044"  Part="1"
+AR Path="/4E388079/4DD1EC8A" Ref="#PWR044"  Part="1"
+F 0 "#PWR044" H 8200 4290 20  0001 C CNN
+F 1 "+5V" H 8200 4290 30  0000 C CNN
+	1    8200 4200
 	1    0    0    -1
 $EndComp
@@
 L POT RV4
 U 1 1 4DD1EC78
-P 7500 3950
+P 8650 4350
 AR Path="/4DEEDDA4/4DD1EC78" Ref="RV4"  Part="1"
 AR Path="/4DEEDD9B/4DD1EC78" Ref="RV3"  Part="1"
@@
 AR Path="/4E1B8870/4DD1EC78" Ref="RV3"  Part="1"
 AR Path="/4E1B886D/4DD1EC78" Ref="RV4"  Part="1"
-F 0 "RV2" H 7500 3850 50  0000 C CNN
-F 1 "POT" H 7500 3950 50  0000 C CNN
-	1    7500 3950
+AR Path="/4E3873D3/4DD1EC78" Ref="RV1"  Part="1"
+AR Path="/4E388079/4DD1EC78" Ref="RV1"  Part="1"
+F 0 "RV1" H 8650 4250 50  0000 C CNN
+F 1 "POT" H 8650 4350 50  0000 C CNN
+	1    8650 4350
 	-1   0    0    1
 $EndComp
@@
 L BUCKPUCK BP4
 U 1 1 4DD1A2DC
-P 4750 3650
+P 5900 4050
 AR Path="/4DEEDDA4/4DD1A2DC" Ref="BP4"  Part="1"
 AR Path="/4DEEDD9B/4DD1A2DC" Ref="BP3"  Part="1"
@@
 AR Path="/4E1B8870/4DD1A2DC" Ref="BP3"  Part="1"
 AR Path="/4E1B886D/4DD1A2DC" Ref="BP4"  Part="1"
-F 0 "BP2" H 5100 3450 60  0000 C CNN
-F 1 "BUCKPUCK" H 4750 3950 60  0000 C CNN
-	1    4750 3650
+AR Path="/4E3873D3/4DD1A2DC" Ref="BP1"  Part="1"
+AR Path="/4E388079/4DD1A2DC" Ref="BP1"  Part="1"
+F 0 "BP1" H 6250 3850 60  0000 C CNN
+F 1 "BUCKPUCK" H 5900 4350 60  0000 C CNN
+	1    5900 4050
 	1    0    0    -1
 $EndComp
@@
 L VAA #PWR43
 U 1 1 4DD1A2DB
-P 3750 3300
+P 4900 3700
 AR Path="/4DEEDDA4/4DD1A2DB" Ref="#PWR43"  Part="1"
 AR Path="/4DEEDD9B/4DD1A2DB" Ref="#PWR36"  Part="1"
@@
 AR Path="/4E1B8870/4DD1A2DB" Ref="#PWR44"  Part="1"
 AR Path="/4E1B886D/4DD1A2DB" Ref="#PWR40"  Part="1"
-F 0 "#PWR36" H 3750 3360 30  0001 C CNN
-F 1 "VAA" H 3750 3410 30  0000 C CNN
-	1    3750 3300
+AR Path="/4E3873D3/4DD1A2DB" Ref="#PWR32"  Part="1"
+AR Path="/4E388079/4DD1A2DB" Ref="#PWR32"  Part="1"
+F 0 "#PWR32" H 4900 3760 30  0001 C CNN
+F 1 "VAA" H 4900 3810 30  0000 C CNN
+	1    4900 3700
 	1    0    0    -1
 $EndComp
@@
 L GND #PWR032
 U 1 1 4DD1A2DA
-P 4250 4100
+P 5400 4500
 AR Path="/4DEEDDA4/4DD1A2DA" Ref="#PWR032"  Part="1"
 AR Path="/4DEEDD9B/4DD1A2DA" Ref="#PWR038"  Part="1"
@@
 AR Path="/4E1B8870/4DD1A2DA" Ref="#PWR036"  Part="1"
 AR Path="/4E1B886D/4DD1A2DA" Ref="#PWR039"  Part="1"
-F 0 "#PWR042" H 4250 4100 30  0001 C CNN
-F 1 "GND" H 4250 4030 30  0001 C CNN
-	1    4250 4100
+AR Path="/4E3873D3/4DD1A2DA" Ref="#PWR045"  Part="1"
+AR Path="/4E388079/4DD1A2DA" Ref="#PWR045"  Part="1"
+F 0 "#PWR045" H 5400 4500 30  0001 C CNN
+F 1 "GND" H 5400 4430 30  0001 C CNN
+	1    5400 4500
 	1    0    0    -1
 $EndComp
@@
 L CONN_2 P12
 U 1 1 4DD1A2D9
-P 6000 3600
+P 7150 4000
 AR Path="/4DEEDDA4/4DD1A2D9" Ref="P12"  Part="1"
 AR Path="/4DEEDD9B/4DD1A2D9" Ref="P11"  Part="1"
@@
 AR Path="/4E1B8870/4DD1A2D9" Ref="P11"  Part="1"
 AR Path="/4E1B886D/4DD1A2D9" Ref="P12"  Part="1"
-F 0 "P10" V 5950 3600 40  0000 C CNN
-F 1 "CurrentOutput" V 6050 3600 40  0000 C CNN
-	1    6000 3600
-	1    0    0    -1
-$EndComp
+AR Path="/4E3873D3/4DD1A2D9" Ref="P9"  Part="1"
+AR Path="/4E388079/4DD1A2D9" Ref="P9"  Part="1"
+F 0 "P9" V 7100 4000 40  0000 C CNN
+F 1 "CurrentOutput" V 7200 4000 40  0000 C CNN
+	1    7150 4000
+	1    0    0    -1
+$EndComp
