File: pcb/buckpuck_current_controller.sch (KiCad schematic (older format))
At the start: 26 parts, among them P1 POWER, P13 BNC, P2 ResetOverride, P3 Display, P4 Switches, P5 CONN_1, P6 CONN_1, P7 CONN_1, P8 CONN_1, U1 V7809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

Commit message: Finished version-4 schematic and board design
Parts:
- removed C4: 0.33uF, symbol C
- removed P2: ResetOverride, symbol CONN_2X2
- removed R1: 68, symbol R
- added C12: 0.1uF, symbol C
- added R6: 150, symbol R
- gave numbers to parts that had none: 1
Connections:
- net D2 is gone; now on net INT_IO: U2.5 (D2(PD2)(INT0))
- net D3 is gone; now on net CS_IO: U2.6 (D3(PD3)(OC2B)(INT1))
- net +5V: now also IO1.18 (Vdd), C12.2, R6.1
- net GND: now also IO1.4 (A1), IO1.5 (A0), IO1.9 (Vss), P4.10, P4.12, P4.14, P4.16, P4.2, P4.4, P4.6, P4.8, C12.1; no longer P4.1, P4.11, P4.13, P4.15, P4.3, P4.5, P4.7, P4.9, P5.1, P6.1, P7.1, P8.1
- net MISO: now also IO1.3 (SO)
- net Switch_A: now also P4.1; no longer P4.2
- net Switch_B: now also P4.3; no longer P4.4
- net Switch_C: now also P4.5; no longer P4.6
- net Switch_D: now also P4.7; no longer P4.8
- net Switch_E: now also P4.13; no longer P4.14
- net Switch_F: now also P4.15; no longer P4.16
- net Switch_Light: now also P4.11; no longer P4.12
- net Switch_Set: now also P4.9; no longer P4.10
- net at IO1.6 (~RESET): now also R6.2
- net CS_IO: now reaches IO1.7 (~CS)
- net INT_IO: now reaches IO1.8 (INT)
- net RST: no longer names the net of U2.3 (RST)
- no-connect marks 15 -> 18
Other:
- moved on the sheet: P4
